File: pcb/lx32-fpga.kicad_pcb (KiCad board)
At the start: 2 copper layers, 80 x 60 mm, 45 parts, among them J1 USB_C_Receptacle_USB2.0_14P, U1 ICE40HX4K-TQ144, U2 AP2112K-3.3, U3 W25Q32JVSS, U4 CH340C, U5 AP2112K-1.2, Y1 Crystal

Commit message: refactor(submission): lx32 full pcb:) (#103)
Parts:
- removed the MH1 at (104.0, 64.0) (x2)
- added C21: 100nF, , F.Cu at (127.0, 62.0)
- added J2: VGA_HDR, , F.Cu at (108.0, 65.0)
- added R5: 68R, , F.Cu at (108.0, 72.0)
- added R6: 68R, , F.Cu at (111.0, 72.0)
- added R7: 68R, , F.Cu at (114.0, 72.0)
- added U6: 23K256, , F.Cu at (120.0, 65.0)
- C1, C10, C11, C12, C2, C3, C4, C5, C6, C7, C8, C9: footprint Capacitor_SMD:C_0402_1005Metric -> C_0402_1005Metric
- C13, C14, C15, C16: footprint Capacitor_SMD:C_0805_2012Metric -> C_0805_2012Metric
- D1, D2: footprint LED_SMD:LED_0805_2012Metric -> LED_0805_2012Metric
- J1: footprint Connector_USB:USB_C_Receptacle_HRO_TYPE-C-31-M-12 -> USB_C_Receptacle
- R1, R2, R3, R4: footprint Resistor_SMD:R_0402_1005Metric -> R_0402_1005Metric
- U1: footprint Package_QFP:TQFP-144_20x20mm_P0.5mm -> TQFP-144_20x20mm_P0.5mm
- U2, U5: footprint Package_TO_SOT_SMD:SOT-23-5 -> SOT-23-5
- U3: footprint Package_SO:SOIC-8_5.3x5.3mm_P1.27mm -> SOIC-8_5.3x5.3mm_P1.27mm
- U4: footprint Package_SO:SOIC-16_3.9x9.9mm_P1.27mm -> SOIC-16_3.9x9.9mm_P1.27mm
- Y1: footprint Crystal:Crystal_SMD_3225-4Pin_3.2x2.5mm -> Crystal_SMD_3225-4Pin
- moved MH1 53.0 mm to (103.0, 117.0)
- moved R1 3.00 mm to (136.0, 109.0)
- moved R2 3.00 mm to (144.0, 109.0)
- moved C15 2.50 mm to (147.5, 113.0)
Connections:
- FID1 pad 1: (no net) -> GND
- FID2 pad 1: (no net) -> GND
Routing:
- net GND: track 209.8 -> 56.0 mm, vias 0 -> 36
- net Net-(U1B-IOR_139): track 42.6 -> 162.1 mm, vias 0 -> 4
- net USB_DP: track 31.1 -> 145.6 mm, vias 0 -> 4
- net VCC_3V3: track 192.7 -> 306.9 mm, vias 0 -> 12
- net Net-(U1B-IOR_147): track 43.1 -> 151.9 mm, vias 0 -> 4
- net SPI_MOSI: track 50.4 -> 131.6 mm, vias 0 -> 4
- net USB_DM: track 30.3 -> 111.2 mm, vias 0 -> 6
- net SPI_MISO: track 60.6 -> 135.7 mm, vias 0 -> 4
- net VCC_1V2: track 100.4 -> 167.4 mm, vias 0 -> 14
- net Net-(U1B-IOR_112): track 36.3 -> 99.2 mm, vias 0 -> 2
- net VBUS: track 50.5 -> 109.3 mm, vias 0 -> 10
- net Net-(U1B-IOR_114): track 34.8 -> 89.5 mm, vias 0 -> 4
- net SPI_CLK: track 53.2 -> 101.6 mm, vias 0 -> 8
- net Net-(U1B-IOR_115): track 42.6 -> 82.3 mm, vias 0 -> 8
- net Net-(U1B-IOR_120): track 42.6 -> 79.2 mm, vias 0 -> 4
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- added copper zone on In1.Cu, net GND
- added copper zone on In2.Cu, net VCC_3V3
- removed copper zone on B.Cu, net GND
- removed copper zone on F.Cu, net GND
Other:
- copper layers 2 -> 4
- board text added: "{dblquote}All we need is love{dblquote}"
